File: backbone.kicad_sch (KiCad schematic)
At the start: 6 parts

Commit message: 0.1v
Ridiculess backbone
Parts:
- removed J?: Borta, LOCAL:PinHeader_2x12_P2.54mm_Vertical, symbol Connector_Generic:Conn_02x12_Top_Bottom
- removed J?: CAM_2, 5_pin_connector:HDRV5W114P0X396_1X5_1974X850X1070P, symbol Connector:Screw_Terminal_01x05
- removed J?: Power, LOCAL:PinHeader_2x12_P2.54mm_Vertical, symbol Connector_Generic:Conn_02x12_Top_Bottom
- removed J?: Sensor, LOCAL:PinHeader_2x12_P2.54mm_Vertical, symbol Connector_Generic:Conn_02x12_Top_Bottom
- removed J?: Communication, LOCAL:PinHeader_2x12_P2.54mm_Vertical, symbol Connector_Generic:Conn_02x12_Top_Bottom
- removed J?: CAM_1, 5_pin_connector:HDRV5W114P0X396_1X5_1974X850X1070P, symbol Connector:Screw_Terminal_01x05
- added J1: Communication, Connector_PinSocket_2.54mm:PinSocket_2x10_P2.54mm_Vertical, symbol Connector_Generic:Conn_02x10_Odd_Even
- added J2: Borta, Connector_PinSocket_2.54mm:PinSocket_2x10_P2.54mm_Vertical, symbol Connector_Generic:Conn_02x10_Odd_Even
- added J3: Power, Connector_PinSocket_2.54mm:PinSocket_2x10_P2.54mm_Vertical, symbol Connector_Generic:Conn_02x10_Odd_Even
Connections:
- net 3.3V: now also J1.17 (Pin_17), J1.18 (Pin_18), J2.17 (Pin_17), J2.18 (Pin_18), J3.17 (Pin_17), J3.18 (Pin_18)
- net 4V: now also J1.3 (Pin_3), J1.4 (Pin_4), J2.3 (Pin_3), J2.4 (Pin_4), J3.3 (Pin_3), J3.4 (Pin_4)
- net GND: now also J1.1 (Pin_1), J1.19 (Pin_19), J1.2 (Pin_2), J1.20 (Pin_20), J2.1 (Pin_1), J2.19 (Pin_19), J2.2 (Pin_2), J2.20 (Pin_20), J3.1 (Pin_1), J3.19 (Pin_19), J3.2 (Pin_2), J3.20 (Pin_20)
- net NC: now also J1.5 (Pin_5), J1.6 (Pin_6), J2.5 (Pin_5), J2.6 (Pin_6), J3.5 (Pin_5), J3.6 (Pin_6)
- new net ADC_3.3V: J2.9 (Pin_9), J3.10 (Pin_10), J3.9 (Pin_9)
- new net ADC_4V: J2.11 (Pin_11), J3.11 (Pin_11), J3.12 (Pin_12)
- new net ADC_VBAT: J2.7 (Pin_7), J3.7 (Pin_7), J3.8 (Pin_8)
- new net BUZZER: J2.15 (Pin_15), J3.15 (Pin_15), J3.16 (Pin_16)
- new net MCU_RX_COM_TX: J1.10 (Pin_10), J1.9 (Pin_9), J2.10 (Pin_10)
- new net MCU_TX_COM_RX: J1.11 (Pin_11), J1.12 (Pin_12), J2.12 (Pin_12)
- new net NC0: J1.7 (Pin_7), J1.8 (Pin_8), J2.8 (Pin_8)
- new net NC1: J1.13 (Pin_13), J1.14 (Pin_14), J2.14 (Pin_14)
- new net NC2: J1.15 (Pin_15), J1.16 (Pin_16), J2.16 (Pin_16)
- new net ROPE_CUT: J2.13 (Pin_13), J3.13 (Pin_13), J3.14 (Pin_14)
- no-connect marks 12 -> 0

Commit message: V1
Parts:
- added H1, H2, H3, H4: M3, MountingHole:MountingHole_3.2mm_M3, symbol Mechanical:MountingHole
Other:
- company: (none) -> BASEMENT
Changed lines of the file:
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@@
 (kicad_sch (version 20211123) (generator eeschema)
   (paper "A4")
+  (title_block
+    (date "%%date%%")
+    (rev "%%version%%")
+    (company "BASEMENT")
+  )
   (wire (pts (xy 104.14 33.02) (xy 101.6 33.02))
     (stroke (width 0) (type default) (color 0 0 0 0))
@@
     (pin "9")
   )
+  (symbol (lib_id "Mechanical:MountingHole") (at 48.26 83.82 0) (unit 1)
+    (in_bom yes) (on_board yes) (fields_autoplaced)
+    (property "Reference" "H4" (id 0) (at 50.8 82.5499 0)
+      (effects (font (size 1.27 1.27)) (justify left))
+    )
+    (property "Value" "M3" (id 1) (at 50.8 85.0899 0)
+      (effects (font (size 1.27 1.27)) (justify left))
+    )
+    (property "Footprint" "MountingHole:MountingHole_3.2mm_M3" (id 2) (at 48.26 83.82 0)
+      (effects (font (size 1.27 1.27)) hide)
+    )
+    (property "Datasheet" "~" (id 3) (at 48.26 83.82 0)
+      (effects (font (size 1.27 1.27)) hide)
+    )
+  )
+  (symbol (lib_id "Mechanical:MountingHole") (at 48.26 77.47 0) (unit 1)
+    (in_bom yes) (on_board yes) (fields_autoplaced)
+    (property "Reference" "H3" (id 0) (at 50.8 76.1999 0)
+      (effects (font (size 1.27 1.27)) (justify left))
+    )
+    (property "Value" "M3" (id 1) (at 50.8 78.7399 0)
+      (effects (font (size 1.27 1.27)) (justify left))
+    )
+    (property "Footprint" "MountingHole:MountingHole_3.2mm_M3" (id 2) (at 48.26 77.47 0)
+      (effects (font (size 1.27 1.27)) hide)
+    )
+    (property "Datasheet" "~" (id 3) (at 48.26 77.47 0)
+      (effects (font (size 1.27 1.27)) hide)
+    )
+  )
   (symbol (lib_id "Connector_Generic:Conn_02x10_Odd_Even") (at 144.78 30.48 0) (unit 1)
     (in_bom yes) (on_board yes) (fields_autoplaced)
@@
     (pin "9")
   )
+  (symbol (lib_id "Mechanical:MountingHole") (at 38.1 77.47 0) (unit 1)
+    (in_bom yes) (on_board yes) (fields_autoplaced)
+    (property "Reference" "H1" (id 0) (at 40.64 76.1999 0)
+      (effects (font (size 1.27 1.27)) (justify left))
+    )
+    (property "Value" "M3" (id 1) (at 40.64 78.7399 0)
+      (effects (font (size 1.27 1.27)) (justify left))
+    )
+    (property "Footprint" "MountingHole:MountingHole_3.2mm_M3" (id 2) (at 38.1 77.47 0)
+      (effects (font (size 1.27 1.27)) hide)
+    )
+    (property "Datasheet" "~" (id 3) (at 38.1 77.47 0)
+      (effects (font (size 1.27 1.27)) hide)
+    )
+  )
+  (symbol (lib_id "Mechanical:MountingHole") (at 38.1 83.82 0) (unit 1)
+    (in_bom yes) (on_board yes) (fields_autoplaced)
+    (property "Reference" "H2" (id 0) (at 40.64 82.5499 0)
+      (effects (font (size 1.27 1.27)) (justify left))
+    )
+    (property "Value" "M3" (id 1) (at 40.64 85.0899 0)
+      (effects (font (size 1.27 1.27)) (justify left))
+    )
+    (property "Footprint" "MountingHole:MountingHole_3.2mm_M3" (id 2) (at 38.1 83.82 0)
+      (effects (font (size 1.27 1.27)) hide)
+    )
+    (property "Datasheet" "~" (id 3) (at 38.1 83.82 0)
+      (effects (font (size 1.27 1.27)) hide)
+    )
+  )
   (symbol (lib_id "Connector_Generic:Conn_02x10_Odd_Even") (at 40.64 30.48 0) (unit 1)
     (in_bom yes) (on_board yes) (fields_autoplaced)
@@
   )
   (symbol_instances
+    (path "/d0ecbb77-ee38-4b93-bb0e-5ef0cfbc7f55"
+      (reference "H1") (unit 1) (value "M3") (footprint "MountingHole:MountingHole_3.2mm_M3")
+    )
+    (path "/dc040eaa-c5dc-4188-a6f2-fc0116f2b706"
+      (reference "H2") (unit 1) (value "M3") (footprint "MountingHole:MountingHole_3.2mm_M3")
+    )
+    (path "/7ee61d4b-0fb9-4e87-8b00-867c083d97d6"
+      (reference "H3") (unit 1) (value "M3") (footprint "MountingHole:MountingHole_3.2mm_M3")
+    )
+    (path "/3bc15bb3-0d23-47bc-9391-774b5766da52"
+      (reference "H4") (unit 1) (value "M3") (footprint "MountingHole:MountingHole_3.2mm_M3")
+    )
     (path "/ebc1575c-0a7f-4019-b729-034e3e047a30"
       (reference "J1") (unit 1) (value "Communication") (footprint "Connector_PinSocket_2.54mm:PinSocket_2x10_P2.54mm_Vertical")
